File: pcb/lupa-breakout.sch (EAGLE design)
At the start: 16 parts

Commit message: more work on breakout
Parts:
- removed CONTROL, POWER: (no value), SparkFun-Connectors:CONN_10"
- added 2.5V_POWER1: (no value), SparkFun-Connectors:CONN_06SILK_FEMALE_PTH
- added 3.3V_POWER, EXPOSURE_CONTROL: (no value), SparkFun-Connectors:CONN_05
- added J1, SPI: 455-1750-1-ND, SparkFun-Connectors:CONN_03
Connections:
- net CLK: now also J1.1; no longer CONTROL.10
- net FRAME_VALID: now also EXPOSURE_CONTROL.4; no longer CONTROL.5
- net GND: now also 2.5V_POWER1.1, 3.3V_POWER.4, J1.3; no longer POWER.10
- net INT_TIME1: now also EXPOSURE_CONTROL.1; no longer CONTROL.8
- net INT_TIME2: now also EXPOSURE_CONTROL.2; no longer CONTROL.7
- net INT_TIME3: now also EXPOSURE_CONTROL.3; no longer CONTROL.6
- net LINE_VALID: now also EXPOSURE_CONTROL.5; no longer CONTROL.4
- net RESET: now also J1.2; no longer CONTROL.9
- net SPI_CLK: now also SPI.2; no longer CONTROL.2
- net SPI_DATA: now also SPI.3; no longer CONTROL.3
- net SPI_EN: now also SPI.1; no longer CONTROL.1
- net VADC: now also 2.5V_POWER1.4; no longer POWER.5
- net VDDA: now also 2.5V_POWER1.5; no longer POWER.7
- net VDDD: now also 2.5V_POWER1.3; no longer POWER.6
- net VDDO: now also 2.5V_POWER1.2; no longer POWER.4
- net VMEM_H: now also 3.3V_POWER.5; no longer POWER.8
- net VPIX: now also 2.5V_POWER1.6; no longer POWER.3
- net VRESET_1: now also 3.3V_POWER.3; no longer POWER.9
- net VRESET_2: now also 3.3V_POWER.2; no longer POWER.2
- net VRESET_3: now also 3.3V_POWER.1; no longer POWER.1
Other:
- moved on the sheet: DATA
