File: pcb/lupa-carrier.brd (EAGLE design)
At the start: 100 x 80 mm, 7 parts, among them IC1 REG1118, IC2 REG1118, IC3 REG1118, IC4 REG1118, IC5 REG1118, IC6 REG1118, IC7 REG1118

Commit message: work on carrier
Parts:
- removed IC1, IC2, IC3, IC4, IC5, IC6, IC7: REG1118, burr-brown:SOT223
- added 2V5_10, 2V5_6, 2V5_7, 2V5_8, 2V5_9, 3V3_3, 3V3_4: REG1118, burr-brown:SOT223
- added IMAGE_DATA: (no value), SparkFun-Connectors:1X10
- added J1, J2: (no value), SparkFun-Connectors:1X08_ROUND
- added J3: (no value), SparkFun-Connectors:1X06
Connections:
- new net CLK: J2.8
- new net D0: IMAGE_DATA.1
- new net D1: IMAGE_DATA.2
- new net D2: IMAGE_DATA.3
- new net D3: IMAGE_DATA.4
- new net D4: IMAGE_DATA.5
- new net D5: IMAGE_DATA.6
- new net D6: IMAGE_DATA.7
- new net D7: IMAGE_DATA.8
- new net D8: IMAGE_DATA.9
- new net D9: IMAGE_DATA.10
- new net FRAME_VALID: J2.2
- new net INT_TIME1: J2.5
- new net INT_TIME2: J2.4
- new net INT_TIME3: J2.3
- new net LINE_VALID: J2.1
- new net RESET: J2.7
- new net SPI_CLK: J1.2
- new net SPI_DATA: J1.3
- new net SPI_EN: J1.1
- new net VADC: 2V5_8.1, J3.4
- new net VDDA: 2V5_7.1, J3.5
- new net VDDD: 2V5_9.1, J3.3
- new net VDDO: 2V5_10.1, J3.2
- new net VIN: 2V5_10.3, 2V5_6.3, 2V5_7.3, 2V5_8.3, 2V5_9.3, 3V3_3.3, 3V3_4.3
- new net VMEM_H: 3V3_3.1, J1.4
- new net VPIX: 2V5_6.1, J3.6
- new net VRESET_1: 3V3_4.1, J1.6
- new net VRESET_2: J1.7
- new net VRESET_3: J1.8
- net GND: now also 2V5_10.2, 2V5_6.2, 2V5_7.2, 2V5_8.2, 2V5_9.2, 3V3_3.2, 3V3_4.2, J1.5, J2.6, J3.1; no longer IC1.2, IC2.2, IC3.2, IC4.2, IC5.2, IC6.2, IC7.2
