File: pcb/lupa300-card.brd (EAGLE design)
At the start: 44.4 x 60.8 mm, 41 parts

Commit message: prog xtal breakout and work on hdmi board
Parts:
- C1, C23, C28, C3: value (none) -> 100uF
- C13, C16, C19, C22, C27: value (none) -> 100nF
- C14, C17, C20, C25, C5: value (none) -> 1nF
- C15, C18, C21, C26, C6: value (none) -> 10nF
- C2, C24, C29, C4: value (none) -> 10uF
