File: pcb/pluto/pluto-camera-trigger-shield.brd (EAGLE design)
At the start: 27.9 x 45.6 mm, 5 parts, among them J3 455-1750-1-ND, K1 694106105102

Commit message: upate trigger shield
Parts:
- added SJ1, SJ2, SJ3, SJ4: (no value), jumper:SJ_2
- moved K1 13.2 mm to (11.4, 43.9), flipped to the top, turned to 270 degrees
- flipped X1 to the top
Connections:
- new net N$3: SJ1.2, X1.3
- new net N$6: SJ2.2, X1.4
- new net N$7: SJ3.2, X1.6
- new net N$8: SJ4.2, X1.8
- net IO10: now also SJ3.3
- net IO12: now also SJ2.1
- net IO13: now also SJ2.3
- net IO3: no longer X1.8
- net IO4: no longer X1.4
- net IO5: now also SJ1.1
- net IO6: now also SJ1.3
- net IO70: now also SJ4.1
- net IO71: now also SJ4.3
- net IO72: no longer X1.6
- net IO73: no longer X1.3
- net IO9: now also SJ3.1
Routing:
- net IO4: track 18.8 -> 0.00 mm
- net VIN: track 63.6 -> 46.3 mm, vias 1 -> 0
- net IO3: track 17.0 -> 0.00 mm
- net N$8: track 0.00 -> 12.4 mm, vias 0 -> 1
- net IO73: track 10.6 -> 0.00 mm
- net IO72: track 9.96 -> 0.00 mm
- net IO12: track 0.00 -> 9.90 mm
- net IO71: track 0.00 -> 9.15 mm
- net IO13: track 0.00 -> 8.85 mm
- net IO9: track 0.00 -> 8.48 mm
- net N$6: track 0.00 -> 8.27 mm, vias 0 -> 1
- net N$7: track 0.00 -> 8.05 mm, vias 0 -> 1
- net N$3: track 0.00 -> 5.86 mm, vias 0 -> 1
- net IO70: track 0.00 -> 4.76 mm
- net IO10: track 0.00 -> 3.64 mm
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