File: pcb/pluto/pluto-camera-trigger-shield.sch (EAGLE design)
At the start: 5 parts, among them J3 455-1750-1-ND, K1 694106105102

Commit message: upate trigger shield
Parts:
- added SJ1, SJ2, SJ3, SJ4: (no value), jumper:SJ2W
Connections:
- new net N$3: SJ1.2, X1.3
- new net N$6: SJ2.2, X1.4
- new net N$7: SJ3.2, X1.6
- new net N$8: SJ4.2, X1.8
- net IO10: now also SJ3.3
- net IO12: now also SJ2.1
- net IO13: now also SJ2.3
- net IO3: no longer X1.8
- net IO4: no longer X1.4
- net IO5: now also SJ1.1
- net IO6: now also SJ1.3
- net IO70: now also SJ4.1
- net IO71: now also SJ4.3
- net IO72: no longer X1.6
- net IO73: no longer X1.3
- net IO9: now also SJ3.1
Other:
- moved on the sheet: X1
Changed lines of the file:
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@@
 <?xml version="1.0" encoding="utf-8"?>
 <!DOCTYPE eagle SYSTEM "eagle.dtd">
-<eagle version="8.5.0">
+<eagle version="8.6.1">
 <drawing>
 <settings>
@@
 <part name="SUPPLY1" library="SparkFun-PowerSymbols" deviceset="VIN" device=""/>
 <part name="J3" library="SparkFun-Connectors" deviceset="CONN_03" device="" value="455-1750-1-ND"/>
+<part name="SJ1" library="jumper" library_urn="urn:adsk.eagle:library:252" deviceset="SJ2W" device="" package3d_urn="urn:adsk.eagle:package:15474/1"/>
+<part name="SJ2" library="jumper" library_urn="urn:adsk.eagle:library:252" deviceset="SJ2W" device="" package3d_urn="urn:adsk.eagle:package:15474/1"/>
+<part name="SJ3" library="jumper" library_urn="urn:adsk.eagle:library:252" deviceset="SJ2W" device="" package3d_urn="urn:adsk.eagle:package:15474/1"/>
+<part name="SJ4" library="jumper" library_urn="urn:adsk.eagle:library:252" deviceset="SJ2W" device="" package3d_urn="urn:adsk.eagle:package:15474/1"/>
 </parts>
 <sheets>
@@
 <instance part="J1" gate="G$1" x="22.86" y="50.8"/>
 <instance part="J2" gate="G$1" x="68.58" y="48.26"/>
-<instance part="X1" gate="G$1" x="58.42" y="12.7"/>
+<instance part="X1" gate="G$1" x="96.52" y="12.7"/>
 <instance part="K1" gate="G$1" x="10.16" y="12.7"/>
 <instance part="GND1" gate="1" x="20.32" y="0"/>
 <instance part="SUPPLY1" gate="G$1" x="20.32" y="20.32"/>
 <instance part="J3" gate="J$1" x="-15.24" y="45.72"/>
+<instance part="SJ1" gate="G$1" x="35.56" y="17.78" rot="R180"/>
+<instance part="SJ2" gate="G$1" x="35.56" y="0" rot="R180"/>
+<instance part="SJ3" gate="G$1" x="35.56" y="-17.78" rot="R180"/>
+<instance part="SJ4" gate="G$1" x="35.56" y="-35.56" rot="R180"/>
 </instances>
 <busses>
@@
 <segment>
 <pinref part="X1" gate="G$1" pin="2"/>
-<wire x1="48.26" y1="20.32" x2="40.64" y2="20.32" width="0.1524" layer="91"/>
-<label x="35.56" y="20.32" size="1.778" layer="95"/>
+<wire x1="86.36" y1="20.32" x2="78.74" y2="20.32" width="0.1524" layer="91"/>
+<label x="73.66" y="20.32" size="1.778" layer="95"/>
 </segment>
 <segment>
 <pinref part="X1" gate="G$1" pin="7"/>
-<wire x1="48.26" y1="7.62" x2="40.64" y2="7.62" width="0.1524" layer="91"/>
-<label x="35.56" y="7.62" size="1.778" layer="95"/>
+<wire x1="86.36" y1="7.62" x2="78.74" y2="7.62" width="0.1524" layer="91"/>
+<label x="73.66" y="7.62" size="1.778" layer="95"/>
 </segment>
 <segment>
@@
 <label x="40.64" y="43.18" size="1.778" layer="95"/>
 </segment>
+<segment>
+<pinref part="SJ4" gate="G$1" pin="1"/>
+<wire x1="35.56" y1="-40.64" x2="35.56" y2="-43.18" width="0.1524" layer="91"/>
+<label x="35.56" y="-43.18" size="1.778" layer="95"/>
+</segment>
 </net>
 <net name="IO71" class="0">
@@
 <label x="40.64" y="40.64" size="1.778" layer="95"/>
 </segment>
+<segment>
+<pinref part="SJ4" gate="G$1" pin="3"/>
+<wire x1="35.56" y1="-30.48" x2="35.56" y2="-27.94" width="0.1524" layer="91"/>
+<label x="35.56" y="-30.48" size="1.778" layer="95"/>
+</segment>
 </net>
 <net name="IO72" class="0">
@@
 <label x="40.64" y="38.1" size="1.778" layer="95"/>
 </segment>
-<segment>
-<pinref part="X1" gate="G$1" pin="6"/>
-<wire x1="48.26" y1="10.16" x2="40.64" y2="10.16" width="0.1524" layer="91"/>
-</segment>
 </net>
 <net name="IO73" class="0">
@@
 <label x="40.64" y="35.56" size="1.778" layer="95"/>
 </segment>
-<segment>
-<pinref part="X1" gate="G$1" pin="3"/>
-<wire x1="48.26" y1="17.78" x2="40.64" y2="17.78" width="0.1524" layer="91"/>
-</segment>
 </net>
 <net name="IO3" class="0">
@@
 <label x="86.36" y="33.02" size="1.778" layer="95"/>
 </segment>
-<segment>
-<pinref part="X1" gate="G$1" pin="8"/>
-<wire x1="48.26" y1="5.08" x2="40.64" y2="5.08" width="0.1524" layer="91"/>
-<label x="35.56" y="5.08" size="1.778" layer="95"/>
-</segment>
 </net>
 <net name="IO4" class="0">
@@
 <label x="86.36" y="35.56" size="1.778" layer="95"/>
 </segment>
-<segment>
-<pinref part="X1" gate="G$1" pin="4"/>
-<wire x1="48.26" y1="15.24" x2="40.64" y2="15.24" width="0.1524" layer="91"/>
-<label x="35.56" y="15.24" size="1.778" layer="95"/>
-</segment>
 </net>
 <net name="IO5" class="0">
@@
 <label x="86.36" y="38.1" size="1.778" layer="95"/>
 </segment>
+<segment>
+<pinref part="SJ1" gate="G$1" pin="1"/>
+<wire x1="35.56" y1="12.7" x2="35.56" y2="10.16" width="0.1524" layer="91"/>
+</segment>
 </net>
 <net name="IO6" class="0">
@@
 <label x="86.36" y="40.64" size="1.778" layer="95"/>
 </segment>
+<segment>
+<pinref part="SJ1" gate="G$1" pin="3"/>
+<wire x1="35.56" y1="22.86" x2="35.56" y2="25.4" width="0.1524" layer="91"/>
+<label x="35.56" y="25.4" size="1.778" layer="95"/>
+</segment>
 </net>
 <net name="IO9" class="0">
@@
 <label x="86.36" y="43.18" size="1.778" layer="95"/>
 </segment>
+<segment>
+<pinref part="SJ3" gate="G$1" pin="1"/>
+<wire x1="35.56" y1="-22.86" x2="35.56" y2="-25.4" width="0.1524" layer="91"/>
+<label x="35.56" y="-25.4" size="1.778" layer="95"/>
+</segment>
 </net>
 <net name="IO10" class="0">
@@
 <label x="86.36" y="45.72" size="1.778" layer="95"/>
 </segment>
+<segment>
+<pinref part="SJ3" gate="G$1" pin="3"/>
+<wire x1="35.56" y1="-12.7" x2="35.56" y2="-10.16" width="0.1524" layer="91"/>
+<label x="35.56" y="-10.16" size="1.778" layer="95"/>
+</segment>
 </net>
 <net name="IO12" class="0">
@@
 <label x="86.36" y="48.26" size="1.778" layer="95"/>
 </segment>
+<segment>
+<pinref part="SJ2" gate="G$1" pin="1"/>
+<wire x1="35.56" y1="-5.08" x2="35.56" y2="-7.62" width="0.1524" layer="91"/>
+<label x="35.56" y="-7.62" size="1.778" layer="95"/>
+</segment>
 </net>
 <net name="IO13" class="0">
@@
 <label x="86.36" y="50.8" size="1.778" layer="95"/>
 </segment>
+<segment>
+<pinref part="SJ2" gate="G$1" pin="3"/>
+<wire x1="35.56" y1="5.08" x2="35.56" y2="7.62" width="0.1524" layer="91"/>
+<label x="35.56" y="7.62" size="1.778" layer="95"/>
+</segment>
 </net>
 <net name="IO15" class="0">
@@
 <segment>
 <pinref part="X1" gate="G$1" pin="1"/>
-<wire x1="48.26" y1="22.86" x2="40.64" y2="22.86" width="0.1524" layer="91"/>
-<label x="35.56" y="22.86" size="1.778" layer="95"/>
+<wire x1="86.36" y1="22.86" x2="78.74" y2="22.86" width="0.1524" layer="91"/>
+<label x="73.66" y="22.86" size="1.778" layer="95"/>
 </segment>
 <segment>
@@
 </segment>
 </net>
+<net name="N$3" class="0">
+<segment>
+<pinref part="SJ1" gate="G$1" pin="2"/>
+<pinref part="X1" gate="G$1" pin="3"/>
+<wire x1="40.64" y1="17.78" x2="86.36" y2="17.78" width="0.1524" layer="91"/>
+</segment>
+</net>
+<net name="N$6" class="0">
+<segment>
+<pinref part="SJ2" gate="G$1" pin="2"/>
+<wire x1="40.64" y1="0" x2="50.8" y2="0" width="0.1524" layer="91"/>
+<wire x1="50.8" y1="0" x2="50.8" y2="15.24" width="0.1524" layer="91"/>
+<pinref part="X1" gate="G$1" pin="4"/>
+<wire x1="50.8" y1="15.24" x2="86.36" y2="15.24" width="0.1524" layer="91"/>
+</segment>
+</net>
+<net name="N$7" class="0">
+<segment>
+<pinref part="SJ3" gate="G$1" pin="2"/>
+<wire x1="40.64" y1="-17.78" x2="53.34" y2="-17.78" width="0.1524" layer="91"/>
+<wire x1="53.34" y1="-17.78" x2="53.34" y2="10.16" width="0.1524" layer="91"/>
+<pinref part="X1" gate="G$1" pin="6"/>
+<wire x1="53.34" y1="10.16" x2="86.36" y2="10.16" width="0.1524" layer="91"/>
+</segment>
+</net>
+<net name="N$8" class="0">
+<segment>
+<pinref part="SJ4" gate="G$1" pin="2"/>
+<wire x1="40.64" y1="-35.56" x2="58.42" y2="-35.56" width="0.1524" layer="91"/>
+<wire x1="58.42" y1="-35.56" x2="58.42" y2="5.08" width="0.1524" layer="91"/>
+<pinref part="X1" gate="G$1" pin="8"/>
+<wire x1="58.42" y1="5.08" x2="86.36" y2="5.08" width="0.1524" layer="91"/>
+</segment>
+</net>
