File: pcb/uZed/lupa-hdmi-carrier.brd (EAGLE design)
At the start: 101.6 x 57.1 mm, 95 parts, among them K1 694108105102

Commit message: added images and silkscreen tweaks on pcb layout. fixed cap lableling.
Parts:
- C22, C23, C26, C27: value (none) -> .1uF
- C24, C25: value .1uf -> .1uF
Changed lines of the file:
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@@
 <layer number="13" name="Route13" color="4" fill="5" visible="no" active="no"/>
 <layer number="14" name="Route14" color="1" fill="6" visible="no" active="no"/>
-<layer number="15" name="Route15" color="58" fill="1" visible="no" active="yes"/>
+<layer number="15" name="Route15" color="58" fill="1" visible="yes" active="yes"/>
 <layer number="16" name="Bottom" color="1" fill="1" visible="yes" active="yes"/>
 <layer number="17" name="Pads" color="2" fill="1" visible="yes" active="yes"/>
@@
 <layer number="21" name="tPlace" color="7" fill="1" visible="yes" active="yes"/>
 <layer number="22" name="bPlace" color="7" fill="1" visible="yes" active="yes"/>
-<layer number="23" name="tOrigins" color="15" fill="1" visible="yes" active="yes"/>
+<layer number="23" name="tOrigins" color="15" fill="1" visible="no" active="yes"/>
 <layer number="24" name="bOrigins" color="15" fill="1" visible="yes" active="yes"/>
 <layer number="25" name="tNames" color="7" fill="1" visible="no" active="yes"/>
-<layer number="26" name="bNames" color="7" fill="1" visible="yes" active="yes"/>
+<layer number="26" name="bNames" color="7" fill="1" visible="no" active="yes"/>
 <layer number="27" name="tValues" color="7" fill="1" visible="no" active="yes"/>
 <layer number="28" name="bValues" color="7" fill="1" visible="no" active="yes"/>
@@
 <layer number="37" name="tTest" color="7" fill="1" visible="no" active="yes"/>
 <layer number="38" name="bTest" color="7" fill="1" visible="no" active="yes"/>
-<layer number="39" name="tKeepout" color="4" fill="11" visible="yes" active="yes"/>
-<layer number="40" name="bKeepout" color="1" fill="11" visible="yes" active="yes"/>
-<layer number="41" name="tRestrict" color="4" fill="10" visible="yes" active="yes"/>
-<layer number="42" name="bRestrict" color="1" fill="10" visible="yes" active="yes"/>
+<layer number="39" name="tKeepout" color="4" fill="11" visible="no" active="yes"/>
+<layer number="40" name="bKeepout" color="1" fill="11" visible="no" active="yes"/>
+<layer number="41" name="tRestrict" color="4" fill="10" visible="no" active="yes"/>
+<layer number="42" name="bRestrict" color="1" fill="10" visible="no" active="yes"/>
 <layer number="43" name="vRestrict" color="2" fill="10" visible="no" active="yes"/>
 <layer number="44" name="Drills" color="7" fill="1" visible="no" active="yes"/>
@@
 <attribute name="SPICEPREFIX" value="R" x="39.0525" y="34.6075" size="1.778" layer="28" rot="MR0" display="off"/>
 </element>
-<element name="C22" library="rcl" library_urn="urn:adsk.eagle:library:334" package="C0603" package3d_urn="urn:adsk.eagle:package:23616/2" value="" x="54.2925" y="40.64" smashed="yes" rot="MR180">
+<element name="C22" library="rcl" library_urn="urn:adsk.eagle:library:334" package="C0603" package3d_urn="urn:adsk.eagle:package:23616/2" value=".1uF" x="54.2925" y="40.64" smashed="yes" rot="MR180">
 <attribute name="NAME" x="57.4675" y="41.275" size="1.27" layer="26" rot="MR180"/>
 <attribute name="SPICEPREFIX" value="C" x="54.2925" y="40.64" size="1.778" layer="28" rot="MR180" display="off"/>
 <attribute name="VALUE" x="53.6575" y="42.545" size="1.27" layer="28" rot="MR180"/>
 </element>
-<element name="C23" library="rcl" library_urn="urn:adsk.eagle:library:334" package="C0603" package3d_urn="urn:adsk.eagle:package:23616/2" value="" x="34.925" y="27.6225" smashed="yes" rot="MR180">
+<element name="C23" library="rcl" library_urn="urn:adsk.eagle:library:334" package="C0603" package3d_urn="urn:adsk.eagle:package:23616/2" value=".1uF" x="34.925" y="27.6225" smashed="yes" rot="MR180">
 <attribute name="NAME" x="34.29" y="43.4975" size="1.27" layer="26" rot="MR180"/>
 <attribute name="SPICEPREFIX" value="C" x="34.925" y="27.6225" size="1.778" layer="28" rot="MR180" display="off"/>
 <attribute name="VALUE" x="34.29" y="29.5275" size="1.27" layer="28" rot="MR180"/>
 </element>
-<element name="C24" library="rcl" library_urn="urn:adsk.eagle:library:334" package="C0603" package3d_urn="urn:adsk.eagle:package:23616/2" value=".1uf" x="39.0525" y="30.7975" smashed="yes" rot="MR180">
+<element name="C24" library="rcl" library_urn="urn:adsk.eagle:library:334" package="C0603" package3d_urn="urn:adsk.eagle:package:23616/2" value=".1uF" x="39.0525" y="30.7975" smashed="yes" rot="MR180">
 <attribute name="NAME" x="40.9575" y="43.4975" size="1.27" layer="26" rot="MR0"/>
 <attribute name="SPICEPREFIX" value="C" x="39.0525" y="30.7975" size="1.778" layer="28" rot="MR180" display="off"/>
 </element>
-<element name="C25" library="rcl" library_urn="urn:adsk.eagle:library:334" package="C0603" package3d_urn="urn:adsk.eagle:package:23616/2" value=".1uf" x="35.2425" y="30.1625" smashed="yes" rot="MR180">
+<element name="C25" library="rcl" library_urn="urn:adsk.eagle:library:334" package="C0603" package3d_urn="urn:adsk.eagle:package:23616/2" value=".1uF" x="35.2425" y="30.1625" smashed="yes" rot="MR180">
 <attribute name="NAME" x="34.29" y="45.085" size="1.27" layer="26" rot="MR180"/>
 <attribute name="SPICEPREFIX" value="C" x="35.2425" y="30.1625" size="1.778" layer="28" rot="MR180" display="off"/>
 </element>
-<element name="C26" library="rcl" library_urn="urn:adsk.eagle:library:334" package="C0603" package3d_urn="urn:adsk.eagle:package:23616/2" value="" x="35.2425" y="32.7025" smashed="yes" rot="MR180">
+<element name="C26" library="rcl" library_urn="urn:adsk.eagle:library:334" package="C0603" package3d_urn="urn:adsk.eagle:package:23616/2" value=".1uF" x="35.2425" y="32.7025" smashed="yes" rot="MR180">
 <attribute name="NAME" x="34.29" y="46.6725" size="1.27" layer="26" rot="MR180"/>
 <attribute name="SPICEPREFIX" value="C" x="35.2425" y="32.7025" size="1.778" layer="28" rot="MR180" display="off"/>
 <attribute name="VALUE" x="34.6075" y="34.6075" size="1.27" layer="28" rot="MR180"/>
 </element>
-<element name="C27" library="rcl" library_urn="urn:adsk.eagle:library:334" package="C0603" package3d_urn="urn:adsk.eagle:package:23616/2" value="" x="39.0525" y="33.3375" smashed="yes" rot="MR180">
+<element name="C27" library="rcl" library_urn="urn:adsk.eagle:library:334" package="C0603" package3d_urn="urn:adsk.eagle:package:23616/2" value=".1uF" x="39.0525" y="33.3375" smashed="yes" rot="MR180">
 <attribute name="NAME" x="40.9575" y="45.085" size="1.27" layer="26" rot="MR180"/>
 <attribute name="SPICEPREFIX" value="C" x="39.0525" y="33.3375" size="1.778" layer="28" rot="MR180" display="off"/>
@@
 </element>
 <element name="C41" library="rcl" library_urn="urn:adsk.eagle:library:334" package="C0603" package3d_urn="urn:adsk.eagle:package:23616/2" value="1uF" x="39.0525" y="21.2725" smashed="yes" rot="MR180">
-<attribute name="NAME" x="40.9575" y="40.3225" size="1.27" layer="26" rot="MR180"/>
+<attribute name="NAME" x="44.45" y="15.875" size="1.27" layer="26" rot="MR0"/>
 <attribute name="SPICEPREFIX" value="C" x="39.0525" y="21.2725" size="1.778" layer="28" rot="MR180" display="off"/>
 </element>
 <element name="C42" library="rcl" library_urn="urn:adsk.eagle:library:334" package="C0603" package3d_urn="urn:adsk.eagle:package:23616/2" value="1uF" x="39.0525" y="22.5425" smashed="yes" rot="MR180">
-<attribute name="NAME" x="40.9575" y="40.3225" size="1.27" layer="26" rot="MR0"/>
+<attribute name="NAME" x="44.45" y="17.4625" size="1.27" layer="26" rot="MR0"/>
 <attribute name="SPICEPREFIX" value="C" x="39.0525" y="22.5425" size="1.778" layer="28" rot="MR180" display="off"/>
 </element>
@@
 </element>
 <element name="C4" library="rcl" library_urn="urn:adsk.eagle:library:334" package="C0603" package3d_urn="urn:adsk.eagle:package:23616/2" value="1uF" x="39.37" y="25.0825" smashed="yes" rot="MR180">
-<attribute name="NAME" x="37.465" y="9.525" size="1.27" layer="26" rot="MR0"/>
+<attribute name="NAME" x="40.9575" y="38.735" size="1.27" layer="26" rot="MR0"/>
 <attribute name="SPICEPREFIX" value="C" x="39.37" y="25.0825" size="1.9304" layer="28" rot="MR180" display="off"/>
 </element>
 <element name="C5" library="rcl" library_urn="urn:adsk.eagle:library:334" package="C0603" package3d_urn="urn:adsk.eagle:package:23616/2" value="1uF" x="39.37" y="26.9875" smashed="yes" rot="MR180">
-<attribute name="NAME" x="37.465" y="11.1125" size="1.27" layer="26" rot="MR0"/>
+<attribute name="NAME" x="40.9575" y="40.3225" size="1.27" layer="26" rot="MR0"/>
 <attribute name="SPICEPREFIX" value="C" x="39.37" y="26.9875" size="1.9304" layer="28" rot="MR180" display="off"/>
 </element>
@@
 </element>
 <element name="U$18" library="lupa300-components" package="XTAL-6PIN" value="SI514" x="35.56" y="15.875" smashed="yes" rot="MR270">
-<attribute name="NAME" x="34.0475" y="12.0275" size="1.778" layer="26" rot="MR180"/>
+<attribute name="NAME" x="35.3175" y="10.44" size="1.778" layer="26" rot="MR180"/>
 </element>
 <element name="C32" library="rcl" library_urn="urn:adsk.eagle:library:334" package="C0603" package3d_urn="urn:adsk.eagle:package:23616/2" value="" x="31.115" y="13.0175" smashed="yes" rot="MR270">
